File: eagle/HUD.sch (EAGLE design)
At the start: 61 parts, among them IC1 ATMEGA644A, IC2 LM2576, J1 AVR_SPI, X1 16 MHz, Y3 4MHz

Commit message: V4 Schematic and board layout
Parts:
- removed D1: 1N5822, diode:SCHOTTKY-DIODEDO201T15
- removed IC2: LM2576, AWJLEagleLib:LM2576S
- removed JP5: DISPLAY, SparkFun-Connectors:M07LOCK
- removed Y3: 4MHz, SparkFun-FreqCtrl:CRYSTALHC49US
- added C17, C18, C20, C23: 0.1uF, SparkFun-Capacitors:560PF-50V-5%(0603)
- added C19: 4.7pF, SparkFun-Capacitors:560PF-50V-5%(0603)
- added C21: 2.2uF, SparkFun-Capacitors:560PF-50V-5%(0603)
- added C22: 2.2uF, resistor:C-EUC1206
- added J2: (no value), SparkFun-Connectors:CONN_20LOCK
- added Q1: 4MHz, crystal:CRYSTALSM49
- added R17, R18, R19: 20K, SparkFun-Passives:RESISTOR0603-RES
- added R20: 1M, SparkFun-Passives:RESISTOR0603-RES
- added R21: 191K, SparkFun-Passives:RESISTOR0603-RES
- added R22: 25.5K, SparkFun-Passives:RESISTOR0603-RES
- added T2, T3: (no value), zetex:NPNSOT323
- added U1, U2, U3, U4: SN74LVC1T45DBVR, MyLibrary:SN74LVC1T45DBVR
- added U5: MCP1825S-3002E/DB, MyLibrary:MCP1825S-3002E/DB
- C13: value 680uF -> 0.1uF; device SparkFun-Capacitors:1000UF-25V(PTH) -> SparkFun-Capacitors:560PF-50V-5%(0603)
- C5: value 100uF -> 47uF; device SparkFun-Capacitors:CAP_POLPTH1 -> resistor:C-EUC1206
- D10, D11: value 7V -> 24V
- L1: value 150uH -> 22uH; device SparkFun-Passives:INDUCTORPWR -> rcl:L-USPIS2816
- R12: value 127K -> 20K
- R16, R6: value 470 -> 34
- U$1: value TPS27082LDDCRDDC6-M -> LT8631; device power:TPS27082LDDCRDDC6-M -> MyLibrary:LT8631
- X1: value 16 MHz -> 10 MHz
Connections:
- removed net DISPLAY_BUSY: IC1.(PCINT4/ADC4)PA4, JP5.4
- removed net EXT_SLEEP: IC1.(PCINT1/ADC1)PA1, JP1.5
- removed net N$26: D6.A, R6.2
- removed net VCC_VFD: JP5.1, U$1.VOUT, U$1.VOUT_2
- removed net VFD_ON: IC1.(PCINT7/ADC7)PA7, U$1.ON/OFF
- removed net VFD_RESET: IC1.(PCINT3/ADC3)PA3, JP5.6
- new net AVR_TO_ELM_3: IC1.(PCINT25/TXD0)PD1, U3.B
- new net C/S_1: IC1.(PCINT6/ADC6)PA6, J2.17
- new net C/S_2: IC1.(PCINT5/ADC5)PA5
- new net D/C: IC1.(PCINT29/OC1A)PD5, J2.4
- new net D0: IC1.(PCINT16/SCL)PC0, J2.7
- new net D1: IC1.(PCINT17/SDA)PC1, J2.8
- new net D2: IC1.(PCINT18/TCK)PC2, J2.9
- new net D3: IC1.(PCINT19/TMS)PC3, J2.10
- new net D4: IC1.(PCINT20/TDO)PC4, J2.11
- new net D5: IC1.(PCINT21/TDI)PC5, J2.12
- new net D6: IC1.(PCINT22/TOSC1)PC6, J2.13
- new net D7: IC1.(PCINT23/TOSC2)PC7, J2.14
- new net E: IC1.(PCINT31/OC2A)PD7, J2.6
- new net ELM_TO_AVR_3: IC1.(PCINT24/RXD0)PD0, U2.A
- new net N$12: C17.1, D10.A, JP1.4, R19.1, T2.B
- new net N$13: C18.1, D11.A, JP1.2, R18.1, T3.B
- new net N$23: C13.2, L1.1, U$1.SW
- new net N$24: C13.1, U$1.BST
- new net N$25: C20.1, U$1.TR/SS
- new net N$27: C19.2, R20.1, R21.2, U$1.FB
- new net N$31: C21.1, U$1.INTVCC
- new net N$34: R22.2, U$1.RT
- new net POWER_CTRL_3: IC1.(PCINT0/ADC0)PA0, U1.A
- new net R/W: IC1.(PCINT30/OC2B/ICP)PD6, J2.5
- new net RES: IC1.(PCINT7/ADC7)PA7, J2.16
- new net RTS_IGNMON_3: IC1.(PCINT1/ADC1)PA1, U4.B
- new net VCC_2: C12.1, C14.2, C15.2, C16.2, C23.2, D12.A, D6.A, IC1.AVCC, IC1.VCC, IC1.VCC@1, IC1.VCC@2, J1.2, J2.19, J2.2, J2.20, R12.2, R14.2, R17.2, U1.VCCA, U2.VCCA, U3.VCCB, U4.VCCB, U5.VOUT
- net AVR_TO_DISPLAY: no longer JP5.2
- net AVR_TO_ELM: now also U3.A; no longer IC1.(PCINT25/TXD0)PD1
- net BTN_LEFT: now also IC1.(PCINT4/ADC4)PA4; no longer IC1.(PCINT21/TDI)PC5
- net BTN_LEFT_EXT: now also R17.1, T2.C; no longer D10.A, JP1.2
- net BTN_RIGHT: now also IC1.(PCINT3/ADC3)PA3; no longer IC1.(PCINT20/TDO)PC4
- net BTN_RIGHT_EXT: now also R12.1, T3.C; no longer D11.A, JP1.4
- net DISPLAY_CLOCK: no longer JP5.5
- net DISPLAY_TO_AVR: no longer JP5.7
- net ELM_TO_AVR: now also U2.B; no longer IC1.(PCINT24/RXD0)PD0
- net GND: now also C17.2, C18.2, C20.2, C21.2, C22.2, C23.1, C5.2, J2.1, R18.2, R19.2, R21.1, R22.1, T2.E, T3.E, U$1.SYNC/MODE, U1.DIR, U1.GND, U2.DIR, U2.GND, U3.DIR, U3.GND, U4.DIR, U4.GND, U5.GND; no longer C13.-, C5.-, D1.A, IC2.!EN, IC2.GND@1, IC2.GND@2, JP5.3
- net IGNMON: now also IC1.(PCINT2/ADC2)PA2; no longer IC1.(PCINT19/TMS)PC3
- net N$1: now also D12.C, R16.1; no longer R12.2, U$1.R1/C1
- net N$10: now also D6.C, R6.1; no longer D12.C, IC1.(PCINT30/OC2B/ICP)PD6
- net N$15: now also Q1.1; no longer Y3.1
- net N$16: now also Q1.2; no longer Y3.2
- net N$4: now also IC1.(PCINT8/XCK0/T0)PB0, R6.2; no longer D6.C, IC1.(PCINT29/OC1A)PD5
- net N$6: now also L1.2, U$1.IND; no longer D1.C, IC2.VO, L1.1
- net N$8: now also IC1.(PCINT9/CLKO/T1)PB1; no longer D12.A
- net POWER_CTRL: now also U1.B; no longer IC1.(PCINT17/SDA)PC1
- net RTS_IGNMON: now also U4.A; no longer IC1.(PCINT18/TCK)PC2
- net VCC: now also C19.1, C5.1, R20.2, U$1.VOUT, U1.VCCB, U2.VCCB, U3.VCCA, U4.VCCA, U5.VIN; no longer C12.1, C13.+, C14.2, C15.2, C16.2, IC1.AVCC, IC1.VCC, IC1.VCC@1, IC1.VCC@2, IC2.FBACK, J1.2, JP1.1, L1.2, R12.1, R14.2, R16.1, R6.1, U$1.VIN
- net V_BATT: now also C22.1, JP1.1, U$1.EN/UV, U$1.VIN; no longer C5.+, IC2.VIN
Other:
- note added: "NHD-3.12-25664UCB2"
- moved on the sheet: C3, C6, C8, D10, D11, D12, D6, JP1, L1, R12, R14, R16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
